File: main.kicad_sch (KiCad schematic)
At the start: 48 parts, among them J1 Conn_01x04, SW1 SW_Push, SW10 SW_Push, SW11 SW_Push, SW12 SW_Push, SW13 SW_Push, SW14 SW_Push, SW15 RotaryEncoder_Switch, SW16 SW_Push, SW17 SW_Push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

Commit message: :construction: (main)
Parts:
- added D21: D, kamo3:Diode_SOD123, symbol Device:D
- added SW21: SW_Push, kamo3:SW_CherryMX_Hotswap_1.00u, symbol Switch:SW_Push
- D1, D10, D11, D12, D13, D14, D2, D3, D4, D5, D6, D7, D8, D9: footprint (none) -> kamo3:Diode_SOD123
- D15: renamed from D16; footprint (none) -> kamo3:Diode_SOD123
- D16: renamed from D17; footprint (none) -> kamo3:Diode_SOD123
- D17: renamed from D18; footprint (none) -> kamo3:Diode_SOD123
- D18: renamed from D19; footprint (none) -> kamo3:Diode_SOD123
- D19: renamed from D20; footprint (none) -> kamo3:Diode_SOD123
- D20: renamed from D15; footprint (none) -> kamo3:Diode_SOD123
- D22: renamed from D26; footprint (none) -> kamo3:Diode_SOD123
- D23: renamed from D27; footprint (none) -> kamo3:Diode_SOD123
- D24: renamed from D28; footprint (none) -> kamo3:Diode_SOD123
- J1: footprint (none) -> kamo3:MJ-4PP-9
- SW1, SW10, SW11, SW12, SW13, SW14, SW2, SW3, SW4, SW5, SW6, SW7, SW8, SW9: footprint (none) -> kamo3:SW_CherryMX_Hotswap_1.00u
- SW15: renamed from SW16; footprint (none) -> kamo3:SW_CherryMX_Hotswap_1.00u
- SW16: renamed from SW17; footprint (none) -> kamo3:SW_CherryMX_Hotswap_1.00u
- SW17: renamed from SW18; footprint (none) -> kamo3:SW_CherryMX_Hotswap_1.00u
- SW18: renamed from SW19; footprint (none) -> kamo3:SW_CherryMX_Hotswap_1.00u
- SW19: renamed from SW20; footprint (none) -> kamo3:SW_CherryMX_Hotswap_1.00u
- SW20: renamed from SW15; footprint (none) -> keebio:RotaryEncoder_EC11
- SW22: renamed from SW27; footprint (none) -> kamo3:SW_CherryMX_Hotswap_1.00u
- SW23: renamed from SW28; footprint (none) -> kamo3:SW_CherryMX_Hotswap_1.00u
- SW24: renamed from SW29; footprint (none) -> kamo3:SW_CherryMX_Hotswap_1.50u
- U1: value ~ -> RP2040_ZERO; footprint (none) -> kamo3:RP2040-ZERO_SMD
Connections:
- net GND: now also U1.22 (GND); no longer U1.31 (GND)
- net VCC: now also U1.23 (VSYS); no longer U1.32 (VSYS)
- net col0: now also U1.3 (GP2); no longer U1.2 (GP2)
- net col1: now also U1.4 (GP3); no longer U1.3 (GP3)
- net col2: now also U1.5 (GP4); no longer U1.4 (GP4)
- net col3: now also U1.6 (GP5), SW21.1; no longer U1.5 (GP5)
- net col4: now also U1.7 (GP6); no longer U1.6 (GP6)
- net col5: now also U1.8 (GP7); no longer U1.7 (GP7)
- net col6: now also SW20.S1, U1.9 (GP8); no longer SW20.S2, U1.8 (GP8)
- net enc_a: now also U1.15 (GP14); no longer U1.9 (GP9)
- net enc_b: now also U1.16 (GP15); no longer U1.10 (GP10)
- net row0: now also U1.10 (GP9); no longer U1.29 (GP29)
- net row1: now also U1.11 (GP10); no longer U1.28 (GP28)
- net row2: now also U1.13 (GP12); no longer U1.27 (GP27)
- net row3: now also U1.14 (GP13), D21.1 (K); no longer U1.26 (GP26)
- net rx: now also U1.1 (GP0); no longer U1.0 (GP0)
- net tx: now also U1.2 (GP1); no longer U1.1 (GP1)
- net at D20.2 (A): now also SW20.S2; no longer SW20.S1
- new net: D21.2 (A), SW21.2
- no-connect marks 16 -> 6
Other:
- moved on the sheet: SW20

Commit message: :construction:
Parts:
- added D25, D26, D27, D28, D29, D30, D31, D32, D33, D34, D35, D36, D37, D38, D39, D40, D41, D42, D43, D44, D45, D46, D47, D48: D, kamo3:Diode_SOD123, symbol Device:D
- added J2: Conn_01x04, kamo3:MJ-4PP-9, symbol Connector_Generic:Conn_01x04
- added SW25, SW26, SW27, SW28, SW29, SW30, SW31, SW32, SW33, SW34, SW35, SW36, SW37, SW38, SW39, SW40, SW41, SW42, SW43, SW45, SW46, SW47: SW_Push, kamo3:SW_CherryMX_Hotswap_1.00u, symbol Switch:SW_Push
- added SW44: RotaryEncoder_Switch, keebio:RotaryEncoder_EC11, symbol Device:RotaryEncoder_Switch
- added SW48: SW_Push, kamo3:SW_CherryMX_Hotswap_1.50u, symbol Switch:SW_Push
- added U2: RP2040_ZERO, kamo3:RP2040-ZERO_SMD, symbol kamo3:RP2040-ZERO
Connections:
- net GND: now also J1.2 (Pin_2), J2.2 (Pin_2), SW44.C, U2.22 (GND); no longer J1.4 (Pin_4)
- net VCC: now also J2.1 (Pin_1), U2.23 (VSYS)
- net rx: now also J1.4 (Pin_4), U1.2 (GP1); no longer J1.3 (Pin_3), U1.1 (GP0)
- removed net tx: J1.2 (Pin_2), U1.2 (GP1)
- new net: D27.2 (A), SW27.2
- new net: D35.2 (A), SW35.2
- new net: D32.2 (A), SW32.2
- new net: D25.2 (A), SW25.2
- new net: D31.2 (A), SW31.2
- new net: D42.2 (A), SW42.2
- new net: D39.2 (A), SW39.2
- new net: D38.2 (A), SW38.2
- new net: D33.2 (A), SW33.2
- new net: D36.2 (A), SW36.2
- new net: D37.2 (A), SW37.2
- new net: D48.2 (A), SW48.2
- new net: D28.2 (A), SW28.2
- new net: D40.2 (A), SW40.2
- new net: D29.2 (A), SW29.2
- new net: D34.2 (A), SW34.2
- new net: D45.2 (A), SW45.2
- new net: D26.2 (A), SW26.2
- new net: D30.2 (A), SW30.2
- new net: D41.2 (A), SW41.2
- new net: D46.2 (A), SW46.2
- new net: D44.2 (A), SW44.S2
- new net: D47.2 (A), SW47.2
- new net: D43.2 (A), SW43.2
- new net col0_r: SW25.1, SW32.1, U2.3 (GP2)
- new net col1_r: SW26.1, SW33.1, SW39.1, U2.4 (GP3)
- new net col2_r: SW27.1, SW34.1, SW40.1, U2.5 (GP4)
- new net col3_r: SW28.1, SW35.1, SW41.1, SW45.1, U2.6 (GP5)
- new net col4_r: SW29.1, SW36.1, SW42.1, SW46.1, U2.7 (GP6)
- new net col5_r: SW30.1, SW37.1, SW43.1, SW47.1, U2.8 (GP7)
- new net col6_r: SW31.1, SW38.1, SW44.S1, SW48.1, U2.9 (GP8)
- new net enc_a_r: SW44.B, U2.15 (GP14)
- new net enc_b_r: SW44.A, U2.16 (GP15)
- new net row0_r: D25.1 (K), D26.1 (K), D27.1 (K), D28.1 (K), D29.1 (K), D30.1 (K), D31.1 (K), U2.10 (GP9)
- new net row1_r: D32.1 (K), D33.1 (K), D34.1 (K), D35.1 (K), D36.1 (K), D37.1 (K), D38.1 (K), U2.11 (GP10)
- new net row2_r: D39.1 (K), D40.1 (K), D41.1 (K), D42.1 (K), D43.1 (K), D44.1 (K), U2.13 (GP12)
- new net row3_r: D45.1 (K), D46.1 (K), D47.1 (K), D48.1 (K), U2.14 (GP13)
- new net rx_r: J2.4 (Pin_4), U2.2 (GP1)
- no-connect marks 6 -> 16

Commit message: :sparkles: (all) PCB assembly is complete
Connections:
- net GND: no longer J2.2 (Pin_2), SW44.C, U2.22 (GND)
- net VCC: no longer J2.1 (Pin_1), U2.23 (VSYS)
- new net GND2: J2.2 (Pin_2), SW44.C, U2.22 (GND)
- new net VCCQ: J2.1 (Pin_1), U2.23 (VSYS)
