File: main.kicad_pcb (KiCad board)
At the start: 2 copper layers, 140.5 x 116 mm, 50 parts, among them J1 Conn_01x04, SW1 SW_Push, SW10 SW_Push, SW11 SW_Push, SW12 SW_Push, SW13 SW_Push, SW14 SW_Push, SW15 SW_Push, SW16 SW_Push, SW17 SW_Push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

Commit message: :construction:
Parts:
- added D25: D, kamo3:Diode_SOD123, B.Cu at (305.8, 63.1)
- added D26: D, kamo3:Diode_SOD123, B.Cu at (286.8, 53.6)
- added D27: D, kamo3:Diode_SOD123, B.Cu at (267.7, 44.1)
- added D28: D, kamo3:Diode_SOD123, B.Cu at (248.7, 39.3)
- added D29: D, kamo3:Diode_SOD123, B.Cu at (229.6, 44.1)
- added D30: D, kamo3:Diode_SOD123, B.Cu at (210.6, 48.9)
- added D31: D, kamo3:Diode_SOD123, B.Cu at (191.5, 58.4)
- added D32: D, kamo3:Diode_SOD123, B.Cu at (305.8, 82.2)
- added D33: D, kamo3:Diode_SOD123, B.Cu at (286.8, 72.7)
- added D34: D, kamo3:Diode_SOD123, B.Cu at (267.7, 63.1)
- added D35: D, kamo3:Diode_SOD123, B.Cu at (248.7, 58.4)
- added D36: D, kamo3:Diode_SOD123, B.Cu at (229.6, 63.1)
- added D37: D, kamo3:Diode_SOD123, B.Cu at (210.6, 67.9)
- added D38: D, kamo3:Diode_SOD123, B.Cu at (191.5, 77.4)
- added D39: D, kamo3:Diode_SOD123, B.Cu at (286.8, 91.7)
- added D40: D, kamo3:Diode_SOD123, B.Cu at (267.7, 82.2)
- added D41: D, kamo3:Diode_SOD123, B.Cu at (248.7, 77.4)
- added D42: D, kamo3:Diode_SOD123, B.Cu at (229.6, 82.2)
- added D43: D, kamo3:Diode_SOD123, B.Cu at (210.6, 87.0)
- added D44: D, kamo3:Diode_SOD123, B.Cu at (210.6, 103.6)
- added D45: D, kamo3:Diode_SOD123, B.Cu at (258.2, 103.6)
- added D46: D, kamo3:Diode_SOD123, B.Cu at (239.1, 103.6)
- added D47: D, kamo3:Diode_SOD123, B.Cu at (214.6, 113.2)
- added D48: D, kamo3:Diode_SOD123, B.Cu at (197.9, 120.3)
- added J2: Conn_01x04, kamo3:MJ-4PP-9, F.Cu at (183.5, 49.5)
- added SW25: SW_Push, kamo3:SW_CherryMX_Hotswap_1.00u, F.Cu at (315.3, 60.8)
- added SW26: SW_Push, kamo3:SW_CherryMX_Hotswap_1.00u, F.Cu at (296.3, 51.2)
- added SW27: SW_Push, kamo3:SW_CherryMX_Hotswap_1.00u, F.Cu at (277.2, 41.7)
- added SW28: SW_Push, kamo3:SW_CherryMX_Hotswap_1.00u, F.Cu at (258.2, 37.0)
- added SW29: SW_Push, kamo3:SW_CherryMX_Hotswap_1.00u, F.Cu at (239.1, 41.7)
- added SW30: SW_Push, kamo3:SW_CherryMX_Hotswap_1.00u, F.Cu at (220.1, 46.5)
- added SW31: SW_Push, kamo3:SW_CherryMX_Hotswap_1.00u, F.Cu at (201.0, 56.0)
- added SW32: SW_Push, kamo3:SW_CherryMX_Hotswap_1.00u, F.Cu at (315.3, 79.8)
- added SW33: SW_Push, kamo3:SW_CherryMX_Hotswap_1.00u, F.Cu at (296.3, 70.3)
- added SW34: SW_Push, kamo3:SW_CherryMX_Hotswap_1.00u, F.Cu at (277.2, 60.8)
- added SW35: SW_Push, kamo3:SW_CherryMX_Hotswap_1.00u, F.Cu at (258.2, 56.0)
- added SW36: SW_Push, kamo3:SW_CherryMX_Hotswap_1.00u, F.Cu at (239.1, 60.8)
- added SW37: SW_Push, kamo3:SW_CherryMX_Hotswap_1.00u, F.Cu at (220.1, 65.5)
- added SW38: SW_Push, kamo3:SW_CherryMX_Hotswap_1.00u, F.Cu at (201.0, 75.1)
- added SW39: SW_Push, kamo3:SW_CherryMX_Hotswap_1.00u, F.Cu at (296.3, 89.3)
- added SW40: SW_Push, kamo3:SW_CherryMX_Hotswap_1.00u, F.Cu at (277.2, 79.8)
- added SW41: SW_Push, kamo3:SW_CherryMX_Hotswap_1.00u, F.Cu at (258.2, 75.1)
- added SW42: SW_Push, kamo3:SW_CherryMX_Hotswap_1.00u, F.Cu at (239.1, 79.8)
- added SW43: SW_Push, kamo3:SW_CherryMX_Hotswap_1.00u, F.Cu at (220.1, 84.6)
- added SW44: RotaryEncoder_Switch, keebio:RotaryEncoder_EC11, F.Cu at (199.8, 95.3)
- added SW45: SW_Push, kamo3:SW_CherryMX_Hotswap_1.00u, F.Cu at (267.7, 101.2)
- added SW46: SW_Push, kamo3:SW_CherryMX_Hotswap_1.00u, F.Cu at (248.7, 101.2)
- added SW47: SW_Push, kamo3:SW_CherryMX_Hotswap_1.00u, F.Cu at (226.0, 107.3)
- added SW48: SW_Push, kamo3:SW_CherryMX_Hotswap_1.50u, F.Cu at (205.5, 121.3)
- added U2: RP2040_ZERO, kamo3:RP2040-ZERO_SMD, F.Cu at (200.5, 32.2)
- moved J1 41.6 mm to (167.5, 49.5), turned to -90 degrees
- moved D1 4.76 mm to (45.2, 63.1)
- moved D10 4.76 mm to (83.3, 63.1)
- moved D12 4.76 mm to (121.4, 63.1)
- moved D13 4.76 mm to (140.4, 67.9)
- moved D14 4.76 mm to (159.5, 77.4)
- moved D15 4.76 mm to (64.2, 91.7)
- moved D16 4.76 mm to (83.3, 82.2)
- moved D17 4.76 mm to (102.3, 77.4)
- moved D18 4.76 mm to (121.4, 82.2)
- moved D19 4.76 mm to (140.4, 87.0)
- moved D21 4.76 mm to (92.8, 103.6)
- moved D22 4.76 mm to (111.9, 103.6)
- moved D4 4.76 mm to (102.3, 39.3)
- moved D6 4.76 mm to (140.4, 48.9)
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Connections:
- J1 pad 2: tx -> GND
- J1 pad 3: rx -> unconnected-(J1-Pin_3-Pad3)
- J1 pad 4: GND -> rx
- U1 pad 1: rx -> unconnected-(U1-GP0-Pad1)
- U1 pad 2: tx -> rx
Routing:
- net VCC: track 106.5 -> 31.2 mm
- net rx: track 12.7 -> 59.0 mm
- net col5_r: track 0.00 -> 38.1 mm
- net col4_r: track 0.00 -> 38.1 mm
- net col2_r: track 0.00 -> 38.1 mm
- net col1_r: track 0.00 -> 38.1 mm
- net col3_r: track 0.00 -> 38.1 mm
- net col6_r: track 0.00 -> 19.0 mm
- net col0_r: track 0.00 -> 19.0 mm
- net col6: track 106.5 -> 87.7 mm, vias 1 -> 0
- net tx: track 17.5 -> 0.00 mm
- net enc_a: track 52.7 -> 70.1 mm, vias 1 -> 0
- net row0: track 208.6 -> 191.4 mm, vias 8 -> 0
- net enc_b: track 62.8 -> 78.2 mm, vias 1 -> 0
- net row2: track 228.2 -> 213.5 mm, vias 8 -> 0
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- added copper zone on B.Cu, net VCC
- added copper zone on F.Cu, net VCC
- removed copper zone on B.Cu, net GND
- removed copper zone on F.Cu, net GND
Other:
- board size 140.5 x 116 mm -> 298.7 x 114.1 mm

Commit message: :sparkles: (all) PCB assembly is complete
Parts:
- moved D47 21.0 mm to (234.4, 106.0)
- moved D48 19.9 mm to (217.7, 122.7)
- moved D43 19.1 mm to (229.6, 86.2)
- moved D28 19.1 mm to (267.7, 39.3)
- moved D35 19.1 mm to (267.7, 58.4)
- moved D41 19.1 mm to (267.7, 77.4)
- moved D26 19.1 mm to (305.8, 53.6)
- moved D30 19.1 mm to (229.6, 48.9)
- moved D33 19.1 mm to (305.8, 72.7)
- moved D37 19.1 mm to (229.6, 67.9)
- moved D39 19.1 mm to (305.8, 91.7)
- moved D45 19.1 mm to (277.2, 103.6)
- moved D29 19.0 mm to (248.7, 44.1)
- moved D31 19.0 mm to (210.6, 58.4)
- moved D36 19.0 mm to (248.7, 63.1)
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Connections:
- J2 pad 1: VCC -> VCCQ
- J2 pad 2: GND -> GND2
- SW44 pad C: GND -> GND2
- U2 pad 22: GND -> GND2
- U2 pad 23: VCC -> VCCQ
Routing:
- net row1_r: track 0.00 -> 216.3 mm, vias 0 -> 9
- net row2_r: track 0.00 -> 207.6 mm, vias 0 -> 8
- net row0_r: track 0.00 -> 198.4 mm, vias 0 -> 8
- net col0_r: track 19.0 -> 201.7 mm, vias 0 -> 1
- net row3_r: track 0.00 -> 169.2 mm, vias 0 -> 3
- net col1_r: track 38.1 -> 192.0 mm, vias 0 -> 1
- net col3_r: track 38.1 -> 169.5 mm, vias 0 -> 1
- net col2_r: track 38.1 -> 162.6 mm, vias 0 -> 1
- net col4_r: track 38.1 -> 147.0 mm, vias 0 -> 1
- net VCCQ: track 0.00 -> 95.4 mm
- net enc_a_r: track 0.00 -> 77.4 mm, vias 0 -> 1
- net enc_b_r: track 0.00 -> 77.2 mm, vias 0 -> 1
- net col6_r: track 19.0 -> 92.9 mm, vias 0 -> 1
- net col5_r: track 38.1 -> 100.7 mm, vias 0 -> 1
- net rx_r: track 0.00 -> 29.5 mm
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- added copper zone on B.Cu, net GND
- added copper zone on F.Cu, net GND
- added copper zone on B.Cu, net GND2
- added copper zone on F.Cu, net GND2
- removed copper zone on B.Cu, net VCC
- removed copper zone on F.Cu, net VCC
Other:
- board size 298.7 x 114.1 mm -> 298.6 x 114.3 mm

Commit message: :construction: (pcb) fix
Parts:
- moved U2 88.6 mm to (288.3, 43.6)
- moved J2 87.9 mm to (271.0, 60.2)
- moved D25 87.7 mm to (409.8, 74.6)
- moved D27 87.7 mm to (374.0, 53.1)
- moved D32 87.7 mm to (409.8, 93.6)
- moved D34 87.7 mm to (374.0, 72.2)
- moved D40 87.7 mm to (374.0, 91.2)
- moved D29 87.7 mm to (335.9, 53.1)
- moved D36 87.7 mm to (335.9, 72.2)
- moved D42 87.7 mm to (335.9, 91.2)
- moved SW29 87.7 mm to (326.4, 50.8)
- moved SW30 87.7 mm to (307.4, 55.5)
- moved SW31 87.7 mm to (288.3, 65.0)
- moved SW36 87.7 mm to (326.4, 69.8)
- moved SW37 87.7 mm to (307.4, 74.6)
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Routing:
- net row1_r: track 216.3 -> 0.00 mm, vias 9 -> 0
- net row2_r: track 207.6 -> 0.00 mm, vias 8 -> 0
- net col0_r: track 201.7 -> 0.00 mm, vias 1 -> 0
- net row0_r: track 198.4 -> 0.00 mm, vias 8 -> 0
- net col1_r: track 192.0 -> 0.00 mm, vias 1 -> 0
- net col3_r: track 169.5 -> 0.00 mm, vias 1 -> 0
- net row3_r: track 169.2 -> 0.00 mm, vias 3 -> 0
- net col2_r: track 162.6 -> 0.00 mm, vias 1 -> 0
- net col4_r: track 147.0 -> 0.00 mm, vias 1 -> 0
- net col5_r: track 100.7 -> 0.00 mm, vias 1 -> 0
- net VCCQ: track 95.4 -> 0.00 mm
- net row3: track 174.3 -> 79.7 mm, vias 1 -> 0
- net col6_r: track 92.9 -> 0.00 mm, vias 1 -> 0
- net row2: track 204.2 -> 123.7 mm, vias 5 -> 6
- net row1: track 231.8 -> 153.0 mm
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- removed copper zone on B.Cu, net GND
- removed copper zone on F.Cu, net GND
- removed copper zone on B.Cu, net GND2
- removed copper zone on F.Cu, net GND2
Other:
- board outline removed

Commit message: :construction: (pcb) write route done.
Parts:
- moved D27 91.0 mm to (283.3, 46.5)
- moved D28 91.0 mm to (264.3, 41.7)
- moved D34 91.0 mm to (283.3, 65.5)
- moved D35 91.0 mm to (264.3, 60.8)
- moved D40 91.0 mm to (283.3, 84.6)
- moved D41 91.0 mm to (264.3, 79.8)
- moved D45 91.0 mm to (273.8, 106.0)
- moved D29 91.0 mm to (245.2, 46.5)
- moved D30 91.0 mm to (226.2, 51.2)
- moved D31 91.0 mm to (207.1, 60.8)
- moved D36 91.0 mm to (245.2, 65.5)
- moved D37 91.0 mm to (226.2, 70.3)
- moved D38 91.0 mm to (207.1, 79.8)
- moved D42 91.0 mm to (245.2, 84.6)
- moved D46 91.0 mm to (254.7, 106.0)
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Routing:
- net row1_r: track 0.00 -> 217.2 mm, vias 0 -> 8
- net row0_r: track 0.00 -> 197.1 mm, vias 0 -> 9
- net row2_r: track 0.00 -> 195.6 mm, vias 0 -> 5
- net col0_r: track 0.00 -> 190.8 mm, vias 0 -> 1
- net col1_r: track 0.00 -> 183.0 mm, vias 0 -> 1
- net col2_r: track 0.00 -> 152.5 mm, vias 0 -> 1
- net col3_r: track 0.00 -> 151.1 mm, vias 0 -> 1
- net row3_r: track 0.00 -> 147.8 mm, vias 0 -> 3
- net col4_r: track 0.00 -> 121.8 mm, vias 0 -> 1
- net col5_r: track 0.00 -> 100.7 mm, vias 0 -> 1
- net row3: track 79.7 -> 173.7 mm, vias 0 -> 1
- net col6_r: track 0.00 -> 86.0 mm, vias 0 -> 1
- net enc_a_r: track 0.00 -> 73.2 mm, vias 0 -> 2
- net enc_b_r: track 0.00 -> 70.9 mm, vias 0 -> 2
- net row2: track 123.7 -> 184.5 mm, vias 6 -> 4
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
Commit message: :bug: (pcb) reconfigure pcb
Parts:
- moved J1 39.9 mm to (133.7, 28.4), turned to 0 degrees
- moved J2 39.3 mm to (215.4, 28.4), turned to 0 degrees
- moved D23 3.10 mm to (134.5, 116.8)
Routing:
- net rx: track 52.8 -> 6.58 mm, vias 1 -> 0
- net rx_r: track 26.6 -> 71.1 mm, vias 0 -> 2
- net VCC: track 25.7 -> 65.7 mm
- net VCCQ: track 48.5 -> 13.4 mm
- net row1: track 202.5 -> 190.3 mm, vias 7 -> 8
- net row2: track 184.5 -> 173.9 mm, vias 4 -> 5
- net col0: track 167.3 -> 159.1 mm
- net row3: track 173.7 -> 167.5 mm
- net col1: track 159.9 -> 155.5 mm
- net row1_r: track 217.2 -> 221.5 mm
- net col2: track 130.9 -> 126.8 mm
- net col5: track 85.6 -> 81.7 mm
- net Net-(D23-A): track 6.89 -> 10.4 mm
- net row2_r: track 195.6 -> 199.1 mm
- net col5_r: track 100.7 -> 97.4 mm
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
Commit message: :sparkles: (all) ready for manufacturing
Parts:
- added G***: LOGO, kamo3:logo, F.Cu at (259.8, 86.3)
- added G***: LOGO, kamo3:logo, F.Cu at (94.8, 86.3)
- moved J2 3.23 mm to (216.3, 25.3)
- moved J1 3.10 mm to (133.7, 25.3)
- moved U2 0.84 mm to (200.8, 34.6)
Routing:
- net rx_r: track 71.1 -> 77.5 mm, vias 2 -> 0
- net VCC: track 65.7 -> 68.8 mm
- net rx: track 6.58 -> 3.98 mm
- net row2_r: track 199.1 -> 196.7 mm
- net row1: track 190.3 -> 192.6 mm
- net col1_r: track 182.4 -> 180.1 mm
- net col0_r: track 190.0 -> 188.0 mm
- net row1_r: track 221.5 -> 219.6 mm
- net enc_b: track 58.7 -> 60.4 mm
- net VCCQ: track 13.4 -> 11.8 mm
- net row2: track 173.9 -> 175.4 mm
- net row0: track 170.3 -> 171.8 mm
- net row3: track 167.5 -> 168.9 mm
- net col3_r: track 150.2 -> 148.9 mm
- net enc_a: track 48.7 -> 49.7 mm
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- added copper zone on B.Cu, net GND
- added copper zone on F.Cu, net GND
- added copper zone on B.Cu, net GND2
- added copper zone on F.Cu, net GND2
Other:
- board outline added: 297.6 x 115.6 mm
