File: plate.kicad_pcb (KiCad board)
At the start: 2 copper layers, 146.8 x 120.4 mm, 0 parts

Commit message: :sparkles: (all) ready for manufacturing
Other:
- board size 146.8 x 120.4 mm -> 142.8 x 115 mm
